File: MicroSwitch-SD-E.kicad_pcb (KiCad board)
At the start: 2 copper layers, 7.7 x 10 mm, 4 parts, among them J1 Conn_01x03_Pin, Q1 BSS84, U1 A3144

Commit message: fix: change 10k to 11k for consistency
Parts:
- R1: value 10k -> 11k
Changed lines of the file:
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@@
 			)
 		)
-		(property "Value" "10k"
+		(property "Value" "11k"
 			(at 0 1.65 90)
 			(layer "F.Fab")
